File: bdpcb.kicad_pcb (KiCad board)
At the start: 2 copper layers, 292 parts, among them K1 KEYSW, K10 KEYSW, K11 KEYSW, K12 KEYSW, K13 KEYSW, K14 KEYSW, K15 KEYSW, K16 KEYSW, K17 KEYSW, K18 KEYSW, K19 KEYSW, K2 KEYSW, K20 KEYSW, K21 KEYSW, K22 KEYSW, K23 KEYSW, K24 KEYSW, K25 KEYSW, K26 KEYSW, K27 KEYSW, K28 KEYSW, K29 KEYSW, K3 KEYSW, K30 KEYSW, K31 KEYSW, K32 KEYSW, K33 KEYSW, K34 KEYSW, K35 KEYSW, K36 KEYSW, K37 KEYSW, K38 KEYSW, K39 KEYSW, K4 KEYSW, K40 KEYSW, K41 KEYSW, K42 KEYSW, K43 KEYSW, K44 KEYSW, K45 KEYSW, K46 KEYSW, K47 KEYSW, K48 KEYSW, K49 KEYSW, K5 KEYSW, K50 KEYSW, K51 KEYSW, K52 KEYSW, K53 KEYSW, K54 KEYSW, K55 KEYSW, K56 KEYSW, K57 KEYSW, K58 KEYSW, K59 KEYSW, K6 KEYSW, K60 KEYSW, K61 KEYSW, K62 KEYSW, K63 KEYSW, K64 KEYSW, K65 KEYSW, K66 KEYSW, K67 KEYSW, K68 KEYSW, K69 KEYSW, K7 KEYSW, K70 KEYSW, K71 KEYSW, K72 KEYSW, K73 KEYSW, K74 KEYSW, K75 KEYSW, K76 KEYSW, K77 KEYSW, K78 KEYSW, K79 KEYSW, K8 KEYSW, K80 KEYSW, K81 KEYSW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

Commit message: changed feather footprint and moving LEDS
Parts:
- moved L29 241.3 mm to (273.1, 50.0)
- moved L13 229.2 mm to (254.0, 31.0)
- moved L15 211.5 mm to (292.1, 31.0)
- moved L30 209.1 mm to (292.1, 50.0)
- moved L20 199.0 mm to (101.6, 50.0)
- moved L70 197.9 mm to (273.0, 107.2)
- moved L18 187.7 mm to (63.5, 50.0)
- moved L75 178.7 mm to (106.4, 126.2)
- moved L74 175.7 mm to (75.4, 126.2)
- moved L68 170.0 mm to (234.9, 107.2)
- moved L16 166.4 mm to (25.4, 50.0)
- moved L50 156.4 mm to (134.9, 88.1)
- moved L39 154.4 mm to (187.3, 69.1)
- moved L62 152.9 mm to (120.6, 107.2)
- moved L24 152.8 mm to (177.8, 50.0)
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
Commit message: LEDs placed
Parts:
- moved L14 198.6 mm to (273.0, 31.0)
- moved L57 184.1 mm to (280.2, 88.1)
- moved L11 156.9 mm to (215.9, 31.0)
- moved L72 153.1 mm to (27.8, 126.2)
- moved L26 140.9 mm to (215.9, 50.0)
- moved L28 134.1 mm to (254.0, 50.0)
- moved L83 128.0 mm to (292.1, 126.2)
- moved L17 126.3 mm to (44.5, 50.0)
- moved L73 123.6 mm to (51.6, 126.2)
- moved L45 118.9 mm to (32.5, 88.1)
- moved L40 116.1 mm to (206.4, 69.1)
- moved L42 111.8 mm to (244.5, 69.1)
- moved L38 109.0 mm to (168.3, 69.1)
- moved L21 101.3 mm to (120.7, 50.0)
- moved L82 101.2 mm to (273.1, 126.2)
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Changed lines of the file:
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@@
   )
   (module QB_RGB_LED_footprint:RGB-REVERSE_MOUNT (layer B.Cu)
-    (at 164.683749 138.5298)
+    (at 292.1 126.21261)
     (fp_text reference L83 (at -2.7235 3.2548) (layer B.SilkS)
       (effects (font (size 0.48 0.48) (thickness 0.15)) (justify mirror))
@@
   )
   (module QB_RGB_LED_footprint:RGB-REVERSE_MOUNT (layer B.Cu)
-    (at 179.363749 164.4598)
+    (at 273.05 126.21261)
     (fp_text reference L82 (at -2.7235 3.2548) (layer B.SilkS)
       (effects (font (size 0.48 0.48) (thickness 0.15)) (justify mirror))
@@
   )
   (module QB_RGB_LED_footprint:RGB-REVERSE_MOUNT (layer B.Cu)
-    (at 109.977499 143.02058)
+    (at 196.85 126.21261)
     (fp_text reference L78 (at -2.7235 3.2548) (layer B.SilkS)
       (effects (font (size 0.48 0.48) (thickness 0.15)) (justify mirror))
@@
   )
   (module QB_RGB_LED_footprint:RGB-REVERSE_MOUNT (layer B.Cu)
-    (at 122.247499 148.75058)
+    (at 137.31875 126.21261)
     (fp_text reference L76 (at -2.7235 3.2548) (layer B.SilkS)
       (effects (font (size 0.48 0.48) (thickness 0.15)) (justify mirror))
@@
   )
   (module QB_RGB_LED_footprint:RGB-REVERSE_MOUNT (layer B.Cu)
-    (at 171.583749 155.7198)
+    (at 51.59375 126.21261)
     (fp_text reference L73 (at -2.7235 3.2548) (layer B.SilkS)
       (effects (font (size 0.48 0.48) (thickness 0.15)) (justify mirror))
@@
   )
   (module QB_RGB_LED_footprint:RGB-REVERSE_MOUNT (layer B.Cu)
-    (at 178.483749 152.9998)
+    (at 27.77875 126.21261)
     (fp_text reference L72 (at -2.7235 3.2548) (layer B.SilkS)
       (effects (font (size 0.48 0.48) (thickness 0.15)) (justify mirror))
@@
   )
   (module QB_RGB_LED_footprint:RGB-REVERSE_MOUNT (layer B.Cu)
-    (at 171.583749 144.2598)
+    (at 254 107.16165)
     (fp_text reference L69 (at -2.7235 3.2548) (layer B.SilkS)
       (effects (font (size 0.48 0.48) (thickness 0.15)) (justify mirror))
@@
   )
   (module QB_RGB_LED_footprint:RGB-REVERSE_MOUNT (layer B.Cu)
-    (at 136.047499 163.22058)
+    (at 215.9 107.16165)
     (fp_text reference L67 (at -2.7235 3.2548) (layer B.SilkS)
       (effects (font (size 0.48 0.48) (thickness 0.15)) (justify mirror))
@@
   )
   (module QB_RGB_LED_footprint:RGB-REVERSE_MOUNT (layer B.Cu)
-    (at 109.977499 137.29058)
+    (at 196.85 107.16165)
     (fp_text reference L66 (at -2.7235 3.2548) (layer B.SilkS)
       (effects (font (size 0.48 0.48) (thickness 0.15)) (justify mirror))
@@
   )
   (module QB_RGB_LED_footprint:RGB-REVERSE_MOUNT (layer B.Cu)
-    (at 115.347499 160.21058)
+    (at 34.9225 107.16165)
     (fp_text reference L58 (at -2.7235 3.2548) (layer B.SilkS)
       (effects (font (size 0.48 0.48) (thickness 0.15)) (justify mirror))
@@
   )
   (module QB_RGB_LED_footprint:RGB-REVERSE_MOUNT (layer B.Cu)
-    (at 108.447499 154.48058)
+    (at 280.19125 88.11069)
     (fp_text reference L57 (at -2.7235 3.2548) (layer B.SilkS)
       (effects (font (size 0.48 0.48) (thickness 0.15)) (justify mirror))
@@
   )
   (module QB_RGB_LED_footprint:RGB-REVERSE_MOUNT (layer B.Cu)
-    (at 157.783749 155.7198)
+    (at 230.185 88.11069)
     (fp_text reference L55 (at -2.7235 3.2548) (layer B.SilkS)
       (effects (font (size 0.48 0.48) (thickness 0.15)) (justify mirror))
@@
   )
   (module QB_RGB_LED_footprint:RGB-REVERSE_MOUNT (layer B.Cu)
-    (at 157.783749 149.9898)
+    (at 192.0875 88.11069)
     (fp_text reference L53 (at -2.7235 3.2548) (layer B.SilkS)
       (effects (font (size 0.48 0.48) (thickness 0.15)) (justify mirror))
@@
   )
   (module QB_RGB_LED_footprint:RGB-REVERSE_MOUNT (layer B.Cu)
-    (at 164.683749 155.7198)
+    (at 173.035 88.11069)
     (fp_text reference L52 (at -2.7235 3.2548) (layer B.SilkS)
       (effects (font (size 0.48 0.48) (thickness 0.15)) (justify mirror))
@@
   )
   (module QB_RGB_LED_footprint:RGB-REVERSE_MOUNT (layer B.Cu)
-    (at 108.447499 148.75058)
+    (at 96.8375 88.11069)
     (fp_text reference L48 (at -2.7235 3.2548) (layer B.SilkS)
       (effects (font (size 0.48 0.48) (thickness 0.15)) (justify mirror))
@@
   )
   (module QB_RGB_LED_footprint:RGB-REVERSE_MOUNT (layer B.Cu)
-    (at 129.147499 157.49058)
+    (at 32.54125 88.11069)
     (fp_text reference L45 (at -2.7235 3.2548) (layer B.SilkS)
       (effects (font (size 0.48 0.48) (thickness 0.15)) (justify mirror))
@@
   )
   (module QB_RGB_LED_footprint:RGB-REVERSE_MOUNT (layer B.Cu)
-    (at 186.263749 164.4598)
+    (at 244.475 69.05973)
     (fp_text reference L42 (at -2.7235 3.2548) (layer B.SilkS)
       (effects (font (size 0.48 0.48) (thickness 0.15)) (justify mirror))
@@
   )
   (module QB_RGB_LED_footprint:RGB-REVERSE_MOUNT (layer B.Cu)
-    (at 171.583749 149.9898)
+    (at 225.425 69.05973)
     (fp_text reference L41 (at -2.7235 3.2548) (layer B.SilkS)
       (effects (font (size 0.48 0.48) (thickness 0.15)) (justify mirror))
@@
   )
   (module QB_RGB_LED_footprint:RGB-REVERSE_MOUNT (layer B.Cu)
-    (at 116.877499 143.02058)
+    (at 206.375 69.05973)
     (fp_text reference L40 (at -2.7235 3.2548) (layer B.SilkS)
       (effects (font (size 0.48 0.48) (thickness 0.15)) (justify mirror))
@@
   )
   (module QB_RGB_LED_footprint:RGB-REVERSE_MOUNT (layer B.Cu)
-    (at 108.447499 160.21058)
+    (at 168.2725 69.05973)
     (fp_text reference L38 (at -2.7235 3.2548) (layer B.SilkS)
       (effects (font (size 0.48 0.48) (thickness 0.15)) (justify mirror))
@@
   )
   (module QB_RGB_LED_footprint:RGB-REVERSE_MOUNT (layer B.Cu)
-    (at 164.683749 149.9898)
+    (at 254 50.00877)
     (fp_text reference L28 (at -2.7235 3.2548) (layer B.SilkS)
       (effects (font (size 0.48 0.48) (thickness 0.15)) (justify mirror))
@@
   )
   (module QB_RGB_LED_footprint:RGB-REVERSE_MOUNT (layer B.Cu)
-    (at 115.347499 148.75058)
+    (at 215.8975 50.00877)
     (fp_text reference L26 (at -2.7235 3.2548) (layer B.SilkS)
       (effects (font (size 0.48 0.48) (thickness 0.15)) (justify mirror))
@@
   )
   (module QB_RGB_LED_footprint:RGB-REVERSE_MOUNT (layer B.Cu)
-    (at 157.783749 144.2598)
+    (at 120.65 50.00877)
     (fp_text reference L21 (at -2.7235 3.2548) (layer B.SilkS)
       (effects (font (size 0.48 0.48) (thickness 0.15)) (justify mirror))
@@
   )
   (module QB_RGB_LED_footprint:RGB-REVERSE_MOUNT (layer B.Cu)
-    (at 115.347499 154.48058)
+    (at 44.45 50.00877)
     (fp_text reference L17 (at -2.7235 3.2548) (layer B.SilkS)
       (effects (font (size 0.48 0.48) (thickness 0.15)) (justify mirror))
@@
   )
   (module QB_RGB_LED_footprint:RGB-REVERSE_MOUNT (layer B.Cu)
-    (at 122.247499 160.21058)
+    (at 273.0475 30.95781)
     (fp_text reference L14 (at -2.7235 3.2548) (layer B.SilkS)
       (effects (font (size 0.48 0.48) (thickness 0.15)) (justify mirror))
@@
   )
   (module QB_RGB_LED_footprint:RGB-REVERSE_MOUNT (layer B.Cu)
-    (at 103.077499 140.01058)
+    (at 215.8975 30.95781)
     (fp_text reference L11 (at -2.7235 3.2548) (layer B.SilkS)
       (effects (font (size 0.48 0.48) (thickness 0.15)) (justify mirror))

Commit message: just diodes left to move, then fine tune and trace
Parts:
- moved TP2 293.1 mm to (8.73, 7.14)
- moved TP3 284.6 mm to (5.56, 26.2)
- moved D68 192.9 mm to (229.3, 104.8)
- moved SW1 184.3 mm to (1.59, 15.1), turned to 90 degrees
- moved U2 181.9 mm to (45.2, 82.6), turned to 180 degrees
- moved TP4 146.5 mm to (151.6, 50.0)
- moved D45 146.2 mm to (26.9, 85.7)
- moved TP5 115.2 mm to (162.7, 82.6)
- moved D61 31.6 mm to (96.0, 104.8)

Commit message: diodes roughly placed
Parts:
- moved TP1 272.4 mm to (29.4, 4.76)
- moved D72 225.9 mm to (22.2, 123.8)
- moved D43 223.0 mm to (258.8, 65.9)
- moved D29 211.3 mm to (266.6, 47.6)
- moved D21 210.4 mm to (115.0, 47.6)
- moved D32 208.9 mm to (49.3, 67.5)
- moved D31 208.8 mm to (24.5, 66.7)
- moved D83 206.2 mm to (286.5, 123.8)
- moved D15 196.5 mm to (285.7, 28.6)
- moved R2 193.4 mm to (18.1, 149.2)
- moved D82 192.9 mm to (267.4, 123.8)
- moved D26 192.4 mm to (210.3, 47.6)
- moved D16 191.7 mm to (20.6, 47.6)
- moved D14 183.3 mm to (267.4, 27.8)
- moved D2 179.8 mm to (38.9, 27.8)
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
Commit message: reverse stabs and outer edge cuts
Parts:
- K75, K77: footprint ai03Footprints:MXOnly-2U-NoLED -> ai03Footprints:MXOnly-2U-ReversedStabilizers-NoLED
- turned U2 to 0 degrees
Other:
- board outline added: 285.8 x 114.3 mm

Commit message: square LED cutouts
Parts:
- turned U4 to 45 degrees

Commit message: beginning diode positioning
Parts:
- moved TP1 17.6 mm to (19.1, 19.1)
- moved D1 15.5 mm to (32.5, 19.8), turned to 270 degrees
- moved D7 15.2 mm to (146.8, 21.4), turned to 90 degrees
- moved D4 15.0 mm to (89.7, 19.8), turned to 270 degrees
- moved D2 15.0 mm to (51.6, 19.8), turned to 270 degrees
- moved D3 14.3 mm to (70.6, 19.8), turned to 270 degrees
- moved D6 13.9 mm to (127.8, 21.4), turned to 90 degrees
- moved D5 13.8 mm to (108.7, 21.4), turned to 90 degrees
- moved U3 1.84 mm to (158.8, 57.4), turned to 45 degrees

Commit message: rounded rectangle holes and starting diode traces
Parts:
- moved D15 15.5 mm to (298.4, 19.8), turned to 270 degrees
- moved D29 15.5 mm to (279.4, 38.9), turned to 270 degrees
- moved D11 14.8 mm to (222.2, 19.8), turned to 270 degrees
- moved D25 14.8 mm to (203.2, 38.9), turned to 270 degrees
- moved D26 14.8 mm to (222.2, 38.9), turned to 270 degrees
- moved D24 14.8 mm to (184.2, 38.9), turned to 270 degrees
- moved D27 14.8 mm to (241.3, 38.9), turned to 270 degrees
- moved D13 14.7 mm to (260.4, 19.8), turned to 270 degrees
- moved D10 14.7 mm to (203.2, 19.8), turned to 270 degrees
- moved D9 14.7 mm to (184.2, 19.8), turned to 270 degrees
- moved D21 14.6 mm to (127.8, 40.5), turned to 180 degrees
- moved D14 14.4 mm to (279.4, 19.8), turned to 270 degrees
- moved D17 14.4 mm to (50.8, 38.9), turned to 270 degrees
- moved D19 14.4 mm to (88.9, 38.9), turned to 270 degrees
- moved D8 14.3 mm to (165.1, 19.8), turned to 270 degrees
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Routing:
- net row0: track 0.00 -> 273.5 mm
- net row1: track 0.00 -> 57.2 mm
- net col0: track 0.00 -> 4.86 mm
- net Net-(D13-Pad2): track 0.00 -> 4.30 mm
- net Net-(D12-Pad2): track 0.00 -> 4.30 mm
- net Net-(D19-Pad2): track 0.00 -> 4.30 mm
- net Net-(D4-Pad2): track 0.00 -> 4.30 mm
- net Net-(D16-Pad2): track 0.00 -> 4.30 mm
- net Net-(D9-Pad2): track 0.00 -> 4.30 mm
- net Net-(D8-Pad2): track 0.00 -> 4.30 mm
- net Net-(D17-Pad2): track 0.00 -> 4.30 mm
- net Net-(D15-Pad2): track 0.00 -> 4.30 mm
- net Net-(D14-Pad2): track 0.00 -> 4.30 mm
- net Net-(D11-Pad2): track 0.00 -> 4.30 mm
- net Net-(D10-Pad2): track 0.00 -> 4.30 mm
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