File: bdpcb.kicad_pcb (KiCad board)
At the start: 2 copper layers, 285.8 x 114.3 mm, 292 parts, among them K1 KEYSW, K10 KEYSW, K11 KEYSW, K12 KEYSW, K13 KEYSW, K14 KEYSW, K15 KEYSW, K16 KEYSW, K17 KEYSW, K18 KEYSW, K19 KEYSW, K2 KEYSW, K20 KEYSW, K21 KEYSW, K22 KEYSW, K23 KEYSW, K24 KEYSW, K25 KEYSW, K26 KEYSW, K27 KEYSW, K28 KEYSW, K29 KEYSW, K3 KEYSW, K30 KEYSW, K31 KEYSW, K32 KEYSW, K33 KEYSW, K34 KEYSW, K35 KEYSW, K36 KEYSW, K37 KEYSW, K38 KEYSW, K39 KEYSW, K4 KEYSW, K40 KEYSW, K41 KEYSW, K42 KEYSW, K43 KEYSW, K44 KEYSW, K45 KEYSW, K46 KEYSW, K47 KEYSW, K48 KEYSW, K49 KEYSW, K5 KEYSW, K50 KEYSW, K51 KEYSW, K52 KEYSW, K53 KEYSW, K54 KEYSW, K55 KEYSW, K56 KEYSW, K57 KEYSW, K58 KEYSW, K59 KEYSW, K6 KEYSW, K60 KEYSW, K61 KEYSW, K62 KEYSW, K63 KEYSW, K64 KEYSW, K65 KEYSW, K66 KEYSW, K67 KEYSW, K68 KEYSW, K69 KEYSW, K7 KEYSW, K70 KEYSW, K71 KEYSW, K72 KEYSW, K73 KEYSW, K74 KEYSW, K75 KEYSW, K76 KEYSW, K77 KEYSW, K78 KEYSW, K79 KEYSW, K8 KEYSW, K80 KEYSW, K81 KEYSW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

Commit message: tidied vertical traces and making superhighway
Parts:
- moved TP5 135.4 mm to (23.0, 101.5)
- moved TP4 134.2 mm to (18.7, 29.8)
- moved D58 3.18 mm to (41.3, 99.2), turned to 180 degrees
Routing:
- net col7: track 107.4 -> 231.4 mm, vias 0 -> 3
- net col6: track 85.2 -> 191.2 mm, vias 0 -> 3
- net col5: track 104.2 -> 193.0 mm, vias 0 -> 3
- net col4: track 84.1 -> 156.7 mm, vias 0 -> 3
- net col3: track 105.1 -> 162.9 mm, vias 0 -> 3
- net row4: track 232.3 -> 261.2 mm, vias 0 -> 2
- net LB_1: track 46.8 -> 53.8 mm
- net Net-(D58-Pad2): track 0.00 -> 3.59 mm
- net LA_1: track 48.6 -> 51.3 mm
- net LB_8: track 49.4 -> 48.4 mm
- net LA_4: track 51.5 -> 52.4 mm
- net LA_7: track 52.8 -> 53.7 mm
- net LA_5: track 51.7 -> 52.5 mm
- net LA_6: track 51.7 -> 52.5 mm
- net LA_10: track 51.8 -> 52.4 mm
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
Commit message: doing LED cols
Parts:
- moved D38 1.59 mm to (174.6, 59.5), turned to 90 degrees
- moved D39 1.59 mm to (193.7, 59.5), turned to 90 degrees
- moved D40 1.59 mm to (212.7, 59.5), turned to 90 degrees
- moved D41 1.59 mm to (231.8, 59.5), turned to 90 degrees
- moved D42 1.59 mm to (250.8, 59.5), turned to 90 degrees
- moved D43 1.59 mm to (269.9, 59.5), turned to 90 degrees
- moved D44 1.59 mm to (293.7, 59.5), turned to 90 degrees
Routing:
- net LA_15: track 25.9 -> 153.7 mm, vias 2 -> 3
- net LA_14: track 53.9 -> 162.8 mm, vias 5 -> 6
- net LA_13: track 51.5 -> 141.5 mm, vias 3 -> 4
- net LA_12: track 52.4 -> 123.6 mm, vias 3 -> 4
- net LA_11: track 52.5 -> 104.8 mm, vias 3 -> 4
- net row2: track 219.1 -> 270.1 mm
- net LA_10: track 52.4 -> 86.0 mm, vias 3 -> 4
- net +3V3: track 4.70 -> 19.8 mm, vias 0 -> 3
- net LA_9: track 52.5 -> 67.0 mm, vias 3 -> 4
- net GND: track 58.2 -> 71.2 mm
- net Net-(C2-Pad1): track 0.00 -> 7.62 mm, vias 0 -> 1
- net row0: track 282.7 -> 281.4 mm
- net LA_8: track 51.5 -> 52.2 mm
Other:
- net class Default: clearance 0.2 -> 0.14
- rule trace_clearance: 0.2 -> 0.14

Commit message: tightening spacing on vias and traces, about to redo it all probs
Parts:
- moved R2 28.1 mm to (133.2, 35.2), turned to 90 degrees
- moved R1 27.4 mm to (135.8, 35.2), turned to 90 degrees
- moved R3 27.3 mm to (128.1, 35.2), turned to 90 degrees
Routing:
- net LA_A: track 324.1 -> 299.5 mm
- net LA_D: track 324.1 -> 310.8 mm
- net +3V3: track 19.8 -> 27.5 mm
- net SDA: track 0.00 -> 1.86 mm
- net SCL: track 0.00 -> 1.86 mm
- net INTB: track 0.00 -> 1.86 mm
- net LA_3: track 52.5 -> 51.9 mm
- net LA_4: track 52.4 -> 51.9 mm

Commit message: deleted all traces and vias
Routing:
- net col14: track 348.2 -> 0.00 mm, vias 1 -> 0
- net LB_G: track 332.2 -> 0.00 mm, vias 32 -> 0
- net col12: track 332.1 -> 0.00 mm, vias 1 -> 0
- net LA_G: track 312.6 -> 0.00 mm, vias 38 -> 0
- net LA_D: track 310.8 -> 0.00 mm, vias 41 -> 0
- net LB_D: track 310.2 -> 0.00 mm, vias 38 -> 0
- net LA_A: track 299.5 -> 0.00 mm, vias 41 -> 0
- net col13: track 299.4 -> 0.00 mm, vias 1 -> 0
- net col11: track 295.9 -> 0.00 mm, vias 1 -> 0
- net LA_C: track 290.6 -> 0.00 mm
- net LA_F: track 290.6 -> 0.00 mm
- net LA_B: track 290.5 -> 0.00 mm
- net LA_E: track 290.5 -> 0.00 mm
- net LB_H: track 286.9 -> 0.00 mm
- net LB_I: track 283.2 -> 0.00 mm
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
Commit message: reoriented diodes
Parts:
- moved D20 8.55 mm to (108.0, 40.5), turned to 180 degrees
- moved D64 7.53 mm to (164.3, 97.6), turned to 90 degrees
- moved D69 1.77 mm to (259.6, 97.6), turned to 90 degrees
- moved D81 1.77 mm to (259.6, 116.7), turned to 90 degrees
- moved D13 1.77 mm to (259.6, 21.4), turned to 90 degrees
- moved D28 1.77 mm to (259.6, 40.5), turned to 90 degrees
- moved D36 1.77 mm to (135.7, 59.5), turned to 90 degrees
- moved D63 1.77 mm to (145.3, 97.6), turned to 90 degrees
- moved D65 1.77 mm to (183.4, 97.6), turned to 90 degrees
- moved D68 1.77 mm to (240.5, 97.6), turned to 90 degrees
- moved D80 1.77 mm to (240.5, 116.7), turned to 90 degrees
- moved D12 1.77 mm to (240.5, 21.4), turned to 90 degrees
- moved D9 1.77 mm to (183.4, 21.4), turned to 90 degrees
- moved D31 1.77 mm to (35.7, 59.5), turned to 90 degrees
- moved D32 1.77 mm to (59.5, 59.5), turned to 90 degrees
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
Commit message: better row/col tracks starting
Routing:
- net LA_F: track 0.00 -> 302.2 mm, vias 0 -> 28
- net LA_C: track 0.00 -> 302.2 mm, vias 0 -> 29
- net LA_I: track 0.00 -> 290.2 mm, vias 0 -> 26
- net LA_D: track 0.00 -> 289.5 mm
- net LA_A: track 0.00 -> 289.4 mm
- net LA_B: track 0.00 -> 289.2 mm
- net LA_E: track 0.00 -> 289.2 mm
- net row0: track 0.00 -> 288.2 mm
- net LA_G: track 0.00 -> 278.4 mm
- net LA_H: track 0.00 -> 278.1 mm
- net row5: track 0.00 -> 275.0 mm
- net row4: track 0.00 -> 269.8 mm
- net row2: track 0.00 -> 229.7 mm
- net row1: track 0.00 -> 220.2 mm
- net row3: track 0.00 -> 212.1 mm
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
Commit message: almost there with row/col tracks
Routing:
- net LB_I: track 0.00 -> 292.9 mm, vias 0 -> 22
- net LB_F: track 0.00 -> 288.2 mm, vias 0 -> 26
- net LB_H: track 0.00 -> 286.8 mm
- net LB_G: track 0.00 -> 282.3 mm
- net LB_E: track 0.00 -> 278.4 mm
- net LB_D: track 0.00 -> 278.3 mm
- net LB_C: track 0.00 -> 247.7 mm, vias 0 -> 23
- net LB_B: track 0.00 -> 218.7 mm
- net LB_A: track 0.00 -> 218.5 mm
- net (no net): track 64.0 -> 0.00 mm, vias 3 -> 0
- net LB_1: track 0.00 -> 58.7 mm, vias 0 -> 3
- net LB_2: track 0.00 -> 28.5 mm, vias 0 -> 3
- net LB_8: track 0.00 -> 27.1 mm, vias 0 -> 3
- net LB_4: track 0.00 -> 26.2 mm, vias 0 -> 3
- net LB_3: track 0.00 -> 26.1 mm, vias 0 -> 3
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
Commit message: idek
Parts:
- turned U3 to 0 degrees
Routing:
- net col8: track 39.0 -> 106.9 mm
- net col1: track 43.5 -> 89.3 mm
- net col11: track 62.9 -> 106.6 mm
- net col9: track 62.9 -> 106.5 mm
- net col10: track 62.9 -> 106.5 mm
- net col0: track 66.4 -> 109.5 mm
- net col5: track 39.5 -> 82.5 mm
- net col12: track 62.9 -> 105.7 mm
- net LA_13: track 24.3 -> 49.7 mm
- net LA_9: track 24.2 -> 49.6 mm
- net LA_12: track 24.2 -> 49.6 mm
- net LA_10: track 24.2 -> 49.6 mm
- net LA_2: track 24.2 -> 49.6 mm
- net LA_11: track 24.2 -> 49.6 mm
- net LA_1: track 27.3 -> 50.8 mm, vias 1 -> 3
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