File: bdpcb.sch (KiCad schematic (older format))
At the start: 298 parts, among them K1 KEYSW, K10 KEYSW, K11 KEYSW, K12 KEYSW, K13 KEYSW, K14 KEYSW, K15 KEYSW, K16 KEYSW, K17 KEYSW, K18 KEYSW, K19 KEYSW, K2 KEYSW, K20 KEYSW, K21 KEYSW, K22 KEYSW, K23 KEYSW, K24 KEYSW, K25 KEYSW, K26 KEYSW, K27 KEYSW, K28 KEYSW, K29 KEYSW, K3 KEYSW, K30 KEYSW, K31 KEYSW, K32 KEYSW, K33 KEYSW, K34 KEYSW, K35 KEYSW, K36 KEYSW, K37 KEYSW, K38 KEYSW, K39 KEYSW, K4 KEYSW, K40 KEYSW, K41 KEYSW, K42 KEYSW, K43 KEYSW, K44 KEYSW, K45 KEYSW, K46 KEYSW, K47 KEYSW, K48 KEYSW, K49 KEYSW, K5 KEYSW, K50 KEYSW, K51 KEYSW, K52 KEYSW, K53 KEYSW, K54 KEYSW, K55 KEYSW, K56 KEYSW, K57 KEYSW, K58 KEYSW, K59 KEYSW, K6 KEYSW, K60 KEYSW, K61 KEYSW, K62 KEYSW, K63 KEYSW, K64 KEYSW, K65 KEYSW, K66 KEYSW, K67 KEYSW, K68 KEYSW, K69 KEYSW, K7 KEYSW, K70 KEYSW, K71 KEYSW, K72 KEYSW, K73 KEYSW, K74 KEYSW, K75 KEYSW, K76 KEYSW, K77 KEYSW, K78 KEYSW, K79 KEYSW, K8 KEYSW, K80 KEYSW, K81 KEYSW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

Commit message: removed led driver addr jumper bridges
Parts:
- removed JP5, JP6, JP8, JP9: 13_bridge, Jumper:SolderJumper-3_P1.3mm_Bridged12_RoundedPad1.0x1.5mm, symbol Jumper:SolderJumper_3_Bridged12
Connections:
- net +3V3: now also U4.43 (ADDR1)
- net GND: now also U3.43 (ADDR1), U3.44 (ADDR2), U4.44 (ADDR2)
Changed lines of the file:
@@
 Wire Wire Line
 	2500 6550 2500 6600
-$Comp
-L Jumper:SolderJumper_3_Bridged12 JP5
-U 1 1 66EA3134
-P 1400 9500
-F 0 "JP5" V 1300 9325 50  0000 L CNN
-F 1 "13_bridge" H 1200 9575 50  0001 L CNN
-F 2 "Jumper:SolderJumper-3_P1.3mm_Bridged12_RoundedPad1.0x1.5mm" H 1400 9500 50  0001 C CNN
-F 3 "~" H 1400 9500 50  0001 C CNN
-	1    1400 9500
-	0    -1   -1   0
-$EndComp
-$Comp
-L Jumper:SolderJumper_3_Bridged12 JP6
-U 1 1 66EA313E
-P 1700 9500
-F 0 "JP6" V 1600 9325 50  0000 L CNN
-F 1 "13_bridge" H 1500 9575 50  0001 L CNN
-F 2 "Jumper:SolderJumper-3_P1.3mm_Bridged12_RoundedPad1.0x1.5mm" H 1700 9500 50  0001 C CNN
-F 3 "~" H 1700 9500 50  0001 C CNN
-	1    1700 9500
-	0    -1   -1   0
-$EndComp
-$Comp
-L Jumper:SolderJumper_3_Bridged12 JP8
-U 1 1 695EC22B
-P 1400 14175
-F 0 "JP8" V 1300 14000 50  0000 L CNN
-F 1 "13_bridge" H 1200 14250 50  0001 L CNN
-F 2 "Jumper:SolderJumper-3_P1.3mm_Bridged12_RoundedPad1.0x1.5mm" H 1400 14175 50  0001 C CNN
-F 3 "~" H 1400 14175 50  0001 C CNN
-	1    1400 14175
-	0    -1   -1   0
-$EndComp
 Wire Wire Line
 	1725 13300 1925 13300
@@
 Wire Wire Line
 	1925 13500 1925 13900
-Wire Wire Line
-	1550 13900 1550 14175
-Wire Wire Line
-	1925 13900 1550 13900
-Wire Wire Line
-	1850 13400 1850 14175
 $Comp
 L power:+3V3 #PWR032
 U 1 1 695EC243
-P 1400 13975
-F 0 "#PWR032" H 1400 13825 50  0001 C CNN
-F 1 "+3V3" H 1375 14125 50  0000 C CNN
-F 2 "" H 1400 13975 50  0001 C CNN
-F 3 "" H 1400 13975 50  0001 C CNN
-	1    1400 13975
-	1    0    0    -1
-$EndComp
-Connection ~ 1700 14375
-Connection ~ 1400 13975
-Wire Wire Line
-	1700 13975 1400 13975
-Wire Wire Line
-	1400 14375 1700 14375
-$Comp
-L Jumper:SolderJumper_3_Bridged12 JP9
-U 1 1 695EC235
-P 1700 14175
-F 0 "JP9" V 1800 14000 50  0000 L CNN
-F 1 "13_bridge" H 1500 14250 50  0001 L CNN
-F 2 "Jumper:SolderJumper-3_P1.3mm_Bridged12_RoundedPad1.0x1.5mm" H 1700 14175 50  0001 C CNN
-F 3 "~" H 1700 14175 50  0001 C CNN
-	1    1700 14175
-	0    -1   1    0
+P 1525 13900
+F 0 "#PWR032" H 1525 13750 50  0001 C CNN
+F 1 "+3V3" H 1500 14050 50  0000 C CNN
+F 2 "" H 1525 13900 50  0001 C CNN
+F 3 "" H 1525 13900 50  0001 C CNN
+	1    1525 13900
+	1    0    0    -1
 $EndComp
 $Comp
 L power:GND #PWR033
 U 1 1 695EC221
-P 1700 14375
-F 0 "#PWR033" H 1700 14125 50  0001 C CNN
-F 1 "GND" H 1700 14200 50  0000 C CNN
-F 2 "" H 1700 14375 50  0001 C CNN
-F 3 "" H 1700 14375 50  0001 C CNN
-	1    1700 14375
+P 1925 13900
+F 0 "#PWR033" H 1925 13650 50  0001 C CNN
+F 1 "GND" H 1925 13725 50  0000 C CNN
+F 2 "" H 1925 13900 50  0001 C CNN
+F 3 "" H 1925 13900 50  0001 C CNN
+	1    1925 13900
 	1    0    0    -1
 $EndComp
@@
 	1725 13650 1725 13600
 Wire Wire Line
-	1550 9225 1550 9500
-Wire Wire Line
-	1925 9225 1550 9225
-Wire Wire Line
-	1925 8825 1925 9225
-Wire Wire Line
-	1850 8725 1850 9500
-Wire Wire Line
 	1925 8725 1850 8725
 Wire Wire Line
-	1725 8925 1725 8975
-$Comp
-L power:+3V3 #PWR021
-U 1 1 66EA3159
-P 1400 9300
-F 0 "#PWR021" H 1400 9150 50  0001 C CNN
-F 1 "+3V3" H 1375 9450 50  0000 C CNN
-F 2 "" H 1400 9300 50  0001 C CNN
-F 3 "" H 1400 9300 50  0001 C CNN
-	1    1400 9300
-	1    0    0    -1
-$EndComp
-Connection ~ 1700 9700
-Connection ~ 1400 9300
-Wire Wire Line
-	1700 9300 1400 9300
-Wire Wire Line
-	1400 9700 1700 9700
-$Comp
-L power:GND #PWR022
-U 1 1 66EA312A
-P 1700 9700
-F 0 "#PWR022" H 1700 9450 50  0001 C CNN
-F 1 "GND" H 1700 9525 50  0000 C CNN
-F 2 "" H 1700 9700 50  0001 C CNN
-F 3 "" H 1700 9700 50  0001 C CNN
-	1    1700 9700
-	1    0    0    -1
-$EndComp
-Wire Wire Line
 	1700 7550 1700 7600
 Connection ~ 1700 7350
@@
 Text Notes 1025 14500 0    50   ~ 0
 slave 1\naddr 1010011X
-Text Notes 1025 9825 0    50   ~ 0
+Text Notes 1350 9200 0    50   ~ 0
 master\naddr 1010000X
 $Comp
@@
 L power:GND #PWR020
 U 1 1 965DA8F2
-P 1725 8975
-F 0 "#PWR020" H 1725 8725 50  0001 C CNN
-F 1 "GND" H 1800 8825 50  0000 R CNN
-F 2 "" H 1725 8975 50  0001 C CNN
-F 3 "" H 1725 8975 50  0001 C CNN
-	1    1725 8975
+P 1725 8925
+F 0 "#PWR020" H 1725 8675 50  0001 C CNN
+F 1 "GND" H 1800 8775 50  0000 R CNN
+F 2 "" H 1725 8925 50  0001 C CNN
+F 3 "" H 1725 8925 50  0001 C CNN
+	1    1725 8925
 	1    0    0    -1
 $EndComp
@@
 Wire Wire Line
 	1825 12400 1925 12400
+Wire Wire Line
+	1850 8725 1850 8925
+Wire Wire Line
+	1850 8925 1725 8925
+Connection ~ 1725 8925
+Wire Wire Line
+	1925 8825 1925 8925
+Wire Wire Line
+	1925 8925 1850 8925
+Connection ~ 1850 8925
+Wire Wire Line
+	1850 13400 1850 13900
+Wire Wire Line
+	1525 13900 1850 13900
 $EndSCHEMATC

Commit message: text sizing up to spec + new labels
Parts:
- renumbered JP14 to JP10, JP15 to JP11, JP10 to JP5, JP11 to JP6, JP12 to JP7, JP7 to JP8, JP13 to JP9, TP2 to TP1, TP1 to TP2
Other:
- note added: "3V3 power\nslide\nswitch"
- note removed: "2.2k i2c pullups\nmay prefer 5.7k?"
- note removed: "power\nslide\nswitch"
